File: hardware/kicad/keyboard.kicad_pcb (KiCad board)
At the start: 2 copper layers, 185 parts, among them SW1 MX, SW10 MX, SW11 MX, SW12 MX, SW13 MX, SW14 MX, SW15 MX, SW16 MX, SW18 MX, SW19 MX, SW2 MX, SW20 MX, SW21 MX, SW22 MX, SW23 MX, SW24 MX, SW25 MX, SW26 MX, SW27 MX, SW28 MX, SW29 MX, SW3 MX, SW30 MX, SW31 MX, SW32 MX, SW33 MX, SW35 MX, SW36 MX, SW37 MX, SW38 MX, SW39 MX, SW4 MX, SW40 MX, SW41 MX, SW42 MX, SW43 MX, SW44 MX, SW45 MX, SW46 MX, SW47 MX, SW48 MX, SW49 MX, SW5 MX, SW50 MX, SW52 MX, SW53 MX, SW54 MX, SW55 MX, SW56 MX, SW57 MX, SW58 MX, SW59 MX, SW6 MX, SW60 MX, SW61 MX, SW62 MX, SW63 MX, SW64 MX, SW65 MX, SW66 MX, SW69 MX, SW7 MX, SW70 MX, SW71 MX, SW72 MX, SW73 MX, SW74 MX, SW75 MX, SW76 MX, SW77 MX, SW78 MX, SW79 MX, SW8 MX, SW80 MX, SW81 MX, SW82 MX, SW83 MX, SW84 MX, SW86 MX, SW87 MX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

Commit message: misc
Parts:
- removed U1: ESP32-S3-WROOM-1, Espressif:ESP32-S3-WROOM-1
- added R10: 0, Resistor_SMD:R_2512_6332Metric_Pad1.40x3.35mm_HandSolder, F.Cu at (180.2, 53.3)
- added R11: 0, Resistor_SMD:R_2512_6332Metric_Pad1.40x3.35mm_HandSolder, F.Cu at (68.5, 61.6)
- added R12: 0, Resistor_SMD:R_2512_6332Metric_Pad1.40x3.35mm_HandSolder, F.Cu at (87.5, 61.6)
- added R13: 0, Resistor_SMD:R_2512_6332Metric_Pad1.40x3.35mm_HandSolder, F.Cu at (106.6, 61.6)
- added R14: 0, Resistor_SMD:R_2512_6332Metric_Pad1.40x3.35mm_HandSolder, F.Cu at (125.6, 64.8)
- added R15: 0, Resistor_SMD:R_2512_6332Metric_Pad1.40x3.35mm_HandSolder, F.Cu at (144.0, 68.6)
- added R16: 0, Resistor_SMD:R_2512_6332Metric_Pad1.40x3.35mm_HandSolder, F.Cu at (165.0, 72.4)
- added R18: 0, Resistor_SMD:R_2512_6332Metric_Pad1.40x3.35mm_HandSolder, F.Cu at (67.8, 80.6)
- added R19: 0, Resistor_SMD:R_2512_6332Metric_Pad1.40x3.35mm_HandSolder, F.Cu at (92.6, 81.9)
- added R20: 0, Resistor_SMD:R_2512_6332Metric_Pad1.40x3.35mm_HandSolder, F.Cu at (112.3, 83.1)
- added R21: 0, Resistor_SMD:R_2512_6332Metric_Pad1.40x3.35mm_HandSolder, F.Cu at (128.1, 85.2)
- added R22: 0, Resistor_SMD:R_2512_6332Metric_Pad1.40x3.35mm_HandSolder, F.Cu at (148.5, 88.1)
- added R23: 0, Resistor_SMD:R_2512_6332Metric_Pad1.40x3.35mm_HandSolder, F.Cu at (166.9, 92.1)
- added R25: 0, Resistor_SMD:R_2512_6332Metric_Pad1.40x3.35mm_HandSolder, F.Cu at (67.2, 99.7)
- added R26: 0, Resistor_SMD:R_2512_6332Metric_Pad1.40x3.35mm_HandSolder, F.Cu at (93.2, 99.7)
- added R27: 0, Resistor_SMD:R_2512_6332Metric_Pad1.40x3.35mm_HandSolder, F.Cu at (112.9, 101.6)
- added R28: 0, Resistor_SMD:R_2512_6332Metric_Pad1.40x3.35mm_HandSolder, F.Cu at (131.3, 104.8)
- added R29: 0, Resistor_SMD:R_2512_6332Metric_Pad1.40x3.35mm_HandSolder, F.Cu at (150.4, 108.0)
- added R30: 0, Resistor_SMD:R_2512_6332Metric_Pad1.40x3.35mm_HandSolder, F.Cu at (168.8, 110.5)
- added R32: 0, Resistor_SMD:R_2512_6332Metric_Pad1.40x3.35mm_HandSolder, F.Cu at (68.5, 118.7)
- added R33: 0, Resistor_SMD:R_2512_6332Metric_Pad1.40x3.35mm_HandSolder, F.Cu at (98.9, 118.7)
- added R34: 0, Resistor_SMD:R_2512_6332Metric_Pad1.40x3.35mm_HandSolder, F.Cu at (117.3, 121.3)
- added R35: 0, Resistor_SMD:R_2512_6332Metric_Pad1.40x3.35mm_HandSolder, F.Cu at (137.0, 125.1)
- added R36: 0, Resistor_SMD:R_2512_6332Metric_Pad1.40x3.35mm_HandSolder, F.Cu at (155.4, 127.6)
- added R38: 0, Resistor_SMD:R_2512_6332Metric_Pad1.40x3.35mm_HandSolder, F.Cu at (238.0, 52.7)
- added R39: 0, Resistor_SMD:R_2512_6332Metric_Pad1.40x3.35mm_HandSolder, F.Cu at (256.4, 48.9)
- added R40: 0, Resistor_SMD:R_2512_6332Metric_Pad1.40x3.35mm_HandSolder, F.Cu at (278.6, 45.7)
- added R41: 0, Resistor_SMD:R_2512_6332Metric_Pad1.40x3.35mm_HandSolder, F.Cu at (297.7, 42.5)
- added R42: 0, Resistor_SMD:R_2512_6332Metric_Pad1.40x3.35mm_HandSolder, F.Cu at (318.0, 39.4)
- added R43: 0, Resistor_SMD:R_2512_6332Metric_Pad1.40x3.35mm_HandSolder, F.Cu at (337.1, 39.4)
- added R44: 0, Resistor_SMD:R_2512_6332Metric_Pad1.40x3.35mm_HandSolder, F.Cu at (359.3, 40.6)
- added R45: 0, Resistor_SMD:R_2512_6332Metric_Pad1.40x3.35mm_HandSolder, F.Cu at (377.7, 39.4)
- added R47: 0, Resistor_SMD:R_2512_6332Metric_Pad1.40x3.35mm_HandSolder, F.Cu at (231.7, 75.6)
- added R48: 0, Resistor_SMD:R_2512_6332Metric_Pad1.40x3.35mm_HandSolder, F.Cu at (250.1, 72.4)
- added R49: 0, Resistor_SMD:R_2512_6332Metric_Pad1.40x3.35mm_HandSolder, F.Cu at (269.8, 69.2)
- added R5: 0, Resistor_SMD:R_2512_6332Metric_Pad1.40x3.35mm_HandSolder, F.Cu at (82.4, 40.8)
- added R50: 0, Resistor_SMD:R_2512_6332Metric_Pad1.40x3.35mm_HandSolder, F.Cu at (288.2, 66.0)
- added R51: 0, Resistor_SMD:R_2512_6332Metric_Pad1.40x3.35mm_HandSolder, F.Cu at (307.9, 61.6)
- added R52: 0, Resistor_SMD:R_2512_6332Metric_Pad1.40x3.35mm_HandSolder, F.Cu at (326.3, 61.6)
- added R53: 0, Resistor_SMD:R_2512_6332Metric_Pad1.40x3.35mm_HandSolder, F.Cu at (339.6, 61.0)
- added R54: 0, Resistor_SMD:R_2512_6332Metric_Pad1.40x3.35mm_HandSolder, F.Cu at (357.4, 61.1)
- added R56: 0, Resistor_SMD:R_2512_6332Metric_Pad1.40x3.35mm_HandSolder, F.Cu at (225.9, 95.2)
- added R57: 0, Resistor_SMD:R_2512_6332Metric_Pad1.40x3.35mm_HandSolder, F.Cu at (245.6, 92.1)
- added R58: 0, Resistor_SMD:R_2512_6332Metric_Pad1.40x3.35mm_HandSolder, F.Cu at (264.7, 87.8)
- added R59: 0, Resistor_SMD:R_2512_6332Metric_Pad1.40x3.35mm_HandSolder, F.Cu at (283.1, 85.1)
- added R6: 0, Resistor_SMD:R_2512_6332Metric_Pad1.40x3.35mm_HandSolder, F.Cu at (101.5, 40.0)
- added R60: 0, Resistor_SMD:R_2512_6332Metric_Pad1.40x3.35mm_HandSolder, F.Cu at (301.5, 81.9)
- added R61: 0, Resistor_SMD:R_2512_6332Metric_Pad1.40x3.35mm_HandSolder, F.Cu at (321.2, 81.3)
- added R62: 0, Resistor_SMD:R_2512_6332Metric_Pad1.40x3.35mm_HandSolder, F.Cu at (340.2, 81.3)
- added R63: 0, Resistor_SMD:R_2512_6332Metric_Pad1.40x3.35mm_HandSolder, F.Cu at (363.7, 81.3)
- added R65: 0, Resistor_SMD:R_2512_6332Metric_Pad1.40x3.35mm_HandSolder, F.Cu at (236.1, 113.0)
- added R66: 0, Resistor_SMD:R_2512_6332Metric_Pad1.40x3.35mm_HandSolder, F.Cu at (253.9, 110.5)
- added R67: 0, Resistor_SMD:R_2512_6332Metric_Pad1.40x3.35mm_HandSolder, F.Cu at (273.6, 106.0)
- added R68: 0, Resistor_SMD:R_2512_6332Metric_Pad1.40x3.35mm_HandSolder, F.Cu at (292.6, 102.9)
- added R69: 0, Resistor_SMD:R_2512_6332Metric_Pad1.40x3.35mm_HandSolder, F.Cu at (311.7, 99.8)
- added R7: 0, Resistor_SMD:R_2512_6332Metric_Pad1.40x3.35mm_HandSolder, F.Cu at (121.2, 42.7)
- added R70: 0, Resistor_SMD:R_2512_6332Metric_Pad1.40x3.35mm_HandSolder, F.Cu at (330.7, 99.1)
- added R71: 0, Resistor_SMD:R_2512_6332Metric_Pad1.40x3.35mm_HandSolder, F.Cu at (340.2, 99.2)
- added R72: 0, Resistor_SMD:R_2512_6332Metric_Pad1.40x3.35mm_HandSolder, F.Cu at (361.8, 99.7)
- added R74: 0, Resistor_SMD:R_2512_6332Metric_Pad1.40x3.35mm_HandSolder, F.Cu at (227.1, 134.0)
- added R76: 0, Resistor_SMD:R_2512_6332Metric_Pad1.40x3.35mm_HandSolder, F.Cu at (264.0, 127.0)
- added R77: 0, Resistor_SMD:R_2512_6332Metric_Pad1.40x3.35mm_HandSolder, F.Cu at (283.1, 123.8)
- added R79: 0, Resistor_SMD:R_2512_6332Metric_Pad1.40x3.35mm_HandSolder, F.Cu at (321.2, 118.7)
- added R8: 0, Resistor_SMD:R_2512_6332Metric_Pad1.40x3.35mm_HandSolder, F.Cu at (141.0, 46.2)
- added R80: 0, Resistor_SMD:R_2512_6332Metric_Pad1.40x3.35mm_HandSolder, F.Cu at (349.8, 118.9)
- added R81: 0, Resistor_SMD:R_2512_6332Metric_Pad1.40x3.35mm_HandSolder, F.Cu at (378.3, 118.7)
- added R9: 0, Resistor_SMD:R_2512_6332Metric_Pad1.40x3.35mm_HandSolder, F.Cu at (163.1, 50.2)
- added ROTARY_SWITCH2: KNOB, Rotary_Encoder:RotaryEncoder_Alps_EC11E-Switch_Vertical_H20mm_CircularMountingHoles, B.Cu at (202.8, 161.8)
- D1, D10, D11, D12, D13, D14, D15, D16, D18, D19, D2, D20, D21, D22, D23, D24, D25, D26, D27, D28, D29, D3, D30, D31, D32, D33, D35, D36, D37, D38, D39, D4, D40, D41, D42, D43, D44, D45, D46, D47, D48, D49, D5, D50, D52, D53, D54, D55, D56, D57, D58, D59, D6, D60, D61, D62, D63, D64, D65, D66, D69, D7, D70, D71, D72, D73, D74, D75, D76, D77, D78, D79, D8, D80, D81, D82, D83, D84, D86, D87, D88, D89, D9, D90, D91, D92, D93, D94, D95, D96, D97, D98: footprint Diode_THT:D_DO-35_SOD27_P7.62mm_Horizontal -> Diode_SMD:D_MiniMELF_Handsoldering
- moved D72 16.5 mm to (106.8, 115.6), turned to 80 degrees
- moved D75 16.5 mm to (163.1, 125.5), turned to 80 degrees
- moved D22 16.5 mm to (114.3, 59.8), turned to 80 degrees
- moved D56 16.5 mm to (120.4, 98.9), turned to 80 degrees
- moved D23 16.5 mm to (133.1, 63.1), turned to 80 degrees
- moved D24 16.5 mm to (151.8, 66.4), turned to 80 degrees
- moved D38 16.5 mm to (100.2, 76.3), turned to 80 degrees
- moved D58 16.5 mm to (157.9, 105.6), turned to 80 degrees
- moved D73 16.5 mm to (125.5, 118.9), turned to 80 degrees
- moved D91 16.5 mm to (165.9, 145.1), turned to 80 degrees
- moved D55 16.5 mm to (101.6, 95.6), turned to 80 degrees
- moved D40 16.5 mm to (137.7, 82.9), turned to 80 degrees
- moved D57 16.5 mm to (139.1, 102.2), turned to 80 degrees
- moved D74 16.5 mm to (144.3, 122.2), turned to 80 degrees
- moved D25 16.5 mm to (170.6, 69.7), turned to 80 degrees
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Connections:
- D1 pad 1: R1 -> LR1
- D10 pad 1: R1 -> RR1
- D11 pad 1: R1 -> RR1
- D12 pad 1: R1 -> RR1
- D13 pad 1: R1 -> RR1
- D14 pad 1: R1 -> RR1
- D15 pad 1: R1 -> RR1
- D16 pad 1: R1 -> RR1
- D18 pad 1: R2 -> LR2
- D19 pad 1: R2 -> LR2
- D2 pad 1: R1 -> LR1
- D20 pad 1: R2 -> LR2
- D21 pad 1: R2 -> LR2
- D22 pad 1: R2 -> LR2
- D23 pad 1: R2 -> LR2
- D24 pad 1: R2 -> LR2
- D25 pad 1: R2 -> LR6
- D26 pad 1: R2 -> RR2
- D27 pad 1: R2 -> RR2
- D28 pad 1: R2 -> RR2
- D29 pad 1: R2 -> RR2
- D3 pad 1: R1 -> LR1
- D30 pad 1: R2 -> RR2
- D31 pad 1: R2 -> RR2
- D32 pad 1: R2 -> RR2
- D33 pad 1: R2 -> RR2
- D35 pad 1: R3 -> LR3
- D36 pad 1: R3 -> LR3
- D37 pad 1: R3 -> LR3
- D38 pad 1: R3 -> LR3
- D39 pad 1: R3 -> LR3
- D4 pad 1: R1 -> LR1
- D40 pad 1: R3 -> LR3
- D41 pad 1: R3 -> LR3
- D42 pad 1: R3 -> RR3
- D43 pad 1: R3 -> RR3
- D44 pad 1: R3 -> RR3
- D45 pad 1: R3 -> RR3
- D46 pad 1: R3 -> RR3
- D47 pad 1: R3 -> RR3
- D48 pad 1: R3 -> RR3
- D49 pad 1: R3 -> RR3
- D5 pad 1: R1 -> LR1
- D50 pad 1: R3 -> RR3
- D52 pad 1: R4 -> LR4
- D53 pad 1: R4 -> LR4
- D54 pad 1: R4 -> LR4
- D55 pad 1: R4 -> LR4
- D56 pad 1: R4 -> LR4
- D57 pad 1: R4 -> LR4
- D58 pad 1: R4 -> LR4
- D59 pad 1: R4 -> RR4
- D6 pad 1: R1 -> LR1
- D60 pad 1: R4 -> RR4
- D61 pad 1: R4 -> RR4
- D62 pad 1: R4 -> RR4
- D63 pad 1: R4 -> RR4
- D64 pad 1: R4 -> RR4
- D65 pad 1: R4 -> RR4
- D66 pad 1: R4 -> RR4
- D69 pad 1: R5 -> LR5
- D7 pad 1: R1 -> LR1
- D70 pad 1: R5 -> LR5
- D71 pad 1: R5 -> LR5
- D72 pad 1: R5 -> LR5
- D73 pad 1: R5 -> LR5
- D74 pad 1: R5 -> LR5
- D75 pad 1: R5 -> LR5
- D76 pad 1: R5 -> RR5
- D77 pad 1: R5 -> RR5
- D78 pad 1: R5 -> RR5
- D79 pad 1: R5 -> RR5
- D8 pad 1: R1 -> RR1
- D80 pad 1: R5 -> RR5
- D81 pad 1: R5 -> RR5
- D82 pad 1: R5 -> RR5
- D83 pad 1: R5 -> RR5
- D84 pad 1: R5 -> RR5
- D86 pad 1: R6 -> LR6
- D87 pad 1: R6 -> LR6
- D88 pad 1: R6 -> LR6
- D89 pad 1: R6 -> LR6
- D9 pad 1: R1 -> RR1
- D90 pad 1: R6 -> LR6
- D91 pad 1: R6 -> LR6
- D92 pad 1: R6 -> RR6
- D93 pad 1: R6 -> RR6
- D94 pad 1: R6 -> RR6
- D95 pad 1: R6 -> RR6
- D96 pad 1: R6 -> RR6
- D97 pad 1: R6 -> RR6
- D98 pad 1: R6 -> RR6
- SW1 pad 1: C1 -> LC1
- SW10 pad 1: unconnected-(SW10-Pad1) -> RC7
- SW11 pad 1: unconnected-(SW11-Pad1) -> RC6
- SW12 pad 1: unconnected-(SW12-Pad1) -> RC5
- SW13 pad 1: unconnected-(SW13-Pad1) -> RC4
- SW14 pad 1: unconnected-(SW14-Pad1) -> RC3
- SW15 pad 1: unconnected-(SW15-Pad1) -> RC2
- SW16 pad 1: unconnected-(SW16-Pad1) -> RC1
- SW18 pad 1: Net-(SW18-Pad1) -> LC1
- SW19 pad 1: C1 -> Net-(R11-Pad1)
- SW2 pad 1: C2 -> LC2
- SW20 pad 1: C2 -> Net-(R12-Pad1)
- SW21 pad 1: C3 -> Net-(R13-Pad1)
- SW22 pad 1: C4 -> Net-(R14-Pad1)
- SW23 pad 1: C5 -> Net-(R15-Pad1)
- SW24 pad 1: C6 -> Net-(R10-Pad2)
- SW25 pad 1: unconnected-(SW25-Pad1) -> Net-(R10-Pad2)
- SW26 pad 1: unconnected-(SW26-Pad1) -> Net-(R38-Pad2)
- SW27 pad 1: unconnected-(SW27-Pad1) -> Net-(R39-Pad2)
- SW28 pad 1: unconnected-(SW28-Pad1) -> Net-(R40-Pad2)
- SW29 pad 1: unconnected-(SW29-Pad1) -> Net-(R41-Pad2)
- SW3 pad 1: C3 -> LC3
- SW30 pad 1: unconnected-(SW30-Pad1) -> Net-(R42-Pad2)
- SW31 pad 1: unconnected-(SW31-Pad1) -> Net-(R43-Pad2)
- SW32 pad 1: unconnected-(SW32-Pad1) -> Net-(R45-Pad2)
- SW33 pad 1: unconnected-(SW33-Pad1) -> RC1
- SW35 pad 1: Net-(SW18-Pad1) -> LC1
- SW36 pad 1: C1 -> Net-(R11-Pad2)
- SW37 pad 1: C2 -> Net-(R12-Pad2)
- SW38 pad 1: C3 -> Net-(R13-Pad2)
- SW39 pad 1: C4 -> Net-(R14-Pad2)
- SW4 pad 1: C4 -> LC4
- SW40 pad 1: C5 -> Net-(R15-Pad2)
- SW41 pad 1: C6 -> Net-(R16-Pad2)
- SW42 pad 1: unconnected-(SW42-Pad1) -> Net-(R47-Pad2)
- SW43 pad 1: unconnected-(SW43-Pad1) -> Net-(R48-Pad2)
- SW44 pad 1: unconnected-(SW44-Pad1) -> Net-(R49-Pad2)
- SW45 pad 1: unconnected-(SW45-Pad1) -> Net-(R50-Pad2)
- SW46 pad 1: unconnected-(SW46-Pad1) -> Net-(R51-Pad2)
- SW47 pad 1: unconnected-(SW47-Pad1) -> Net-(R52-Pad2)
- SW48 pad 1: unconnected-(SW48-Pad1) -> Net-(R53-Pad2)
- SW49 pad 1: unconnected-(SW49-Pad1) -> Net-(R54-Pad2)
- SW5 pad 1: C5 -> LC5
- SW50 pad 1: unconnected-(SW50-Pad1) -> RC1
- SW52 pad 1: Net-(SW18-Pad1) -> LC1
- SW53 pad 1: C1 -> Net-(R18-Pad2)
- SW54 pad 1: C2 -> Net-(R19-Pad2)
- SW55 pad 1: C3 -> Net-(R20-Pad2)
- SW56 pad 1: C4 -> Net-(R21-Pad2)
- SW57 pad 1: C5 -> Net-(R22-Pad2)
- SW58 pad 1: C6 -> Net-(R23-Pad2)
- SW59 pad 1: unconnected-(SW59-Pad1) -> Net-(R56-Pad2)
- SW6 pad 1: C6 -> LC6
- SW60 pad 1: unconnected-(SW60-Pad1) -> Net-(R57-Pad2)
- SW61 pad 1: unconnected-(SW61-Pad1) -> Net-(R58-Pad2)
- SW62 pad 1: unconnected-(SW62-Pad1) -> Net-(R59-Pad2)
- SW63 pad 1: unconnected-(SW63-Pad1) -> Net-(R60-Pad2)
- SW64 pad 1: unconnected-(SW64-Pad1) -> Net-(R61-Pad2)
- SW65 pad 1: unconnected-(SW65-Pad1) -> Net-(R63-Pad2)
- SW66 pad 1: unconnected-(SW66-Pad1) -> RC1
- SW69 pad 1: Net-(SW18-Pad1) -> LC1
- SW7 pad 1: unconnected-(SW7-Pad1) -> LC7
- SW70 pad 1: C1 -> Net-(R25-Pad2)
- SW71 pad 1: C2 -> Net-(R26-Pad2)
- SW72 pad 1: C3 -> Net-(R27-Pad2)
- SW73 pad 1: C4 -> Net-(R28-Pad2)
- SW74 pad 1: C5 -> Net-(R29-Pad2)
- SW75 pad 1: C6 -> Net-(R30-Pad2)
- SW76 pad 1: unconnected-(SW76-Pad1) -> Net-(R65-Pad2)
- SW77 pad 1: unconnected-(SW77-Pad1) -> Net-(R66-Pad2)
- SW78 pad 1: unconnected-(SW78-Pad1) -> Net-(R67-Pad2)
- SW79 pad 1: unconnected-(SW79-Pad1) -> Net-(R68-Pad2)
- SW8 pad 1: unconnected-(SW8-Pad1) -> RC9
- SW80 pad 1: unconnected-(SW80-Pad1) -> Net-(R69-Pad2)
- SW81 pad 1: unconnected-(SW81-Pad1) -> Net-(R70-Pad2)
- SW82 pad 1: unconnected-(SW82-Pad1) -> Net-(R71-Pad2)
- SW83 pad 1: unconnected-(SW83-Pad1) -> Net-(R72-Pad2)
- SW84 pad 1: unconnected-(SW84-Pad1) -> RC1
- SW86 pad 1: Net-(SW18-Pad1) -> LC1
- SW87 pad 1: C1 -> Net-(R32-Pad2)
- SW88 pad 1: C2 -> Net-(R33-Pad2)
- SW89 pad 1: C3 -> Net-(R34-Pad2)
- SW9 pad 1: unconnected-(SW9-Pad1) -> RC8
- SW90 pad 1: C4 -> Net-(R35-Pad2)
- SW91 pad 1: C5 -> Net-(R36-Pad2)
- SW92 pad 1: unconnected-(SW92-Pad1) -> Net-(R74-Pad2)
- SW93 pad 1: unconnected-(SW93-Pad1) -> Net-(R76-Pad2)
- SW94 pad 1: unconnected-(SW94-Pad1) -> Net-(R77-Pad2)
- SW95 pad 1: unconnected-(SW95-Pad1) -> Net-(R79-Pad2)
- SW96 pad 1: unconnected-(SW96-Pad1) -> Net-(R80-Pad2)
- SW97 pad 1: unconnected-(SW97-Pad1) -> Net-(R81-Pad2)
- SW98 pad 1: unconnected-(SW98-Pad1) -> RC1
Routing:
- net LC1: track 0.00 -> 195.9 mm
- net RR3: track 0.00 -> 177.7 mm
- net RR5: track 0.00 -> 177.5 mm
- net RR2: track 0.00 -> 170.4 mm
- net RR4: track 0.00 -> 166.1 mm
- net RR1: track 0.00 -> 164.7 mm
- net RR6: track 0.00 -> 159.6 mm
- net LR6: track 0.00 -> 146.0 mm
- net LR5: track 0.00 -> 142.7 mm
- net LR4: track 0.00 -> 137.7 mm
- net LR3: track 0.00 -> 136.4 mm
- net LR2: track 0.00 -> 131.3 mm
- net RC1: track 0.00 -> 124.8 mm
- net LR1: track 0.00 -> 124.7 mm
- net Net-(R10-Pad2): track 0.00 -> 36.7 mm
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
Commit message: misc
Parts:
- moved R61 0.76 mm to (321.2, 80.5)
Routing:
- net Net-(D98-A): track 0.00 -> 7.05 mm
- net Net-(R57-Pad2): track 26.7 -> 19.8 mm
- net LC1: track 195.9 -> 202.8 mm
- net Net-(R23-Pad2): track 6.76 -> 12.9 mm
- net Net-(R52-Pad2): track 16.8 -> 15.3 mm
- net Net-(R53-Pad2): track 14.5 -> 13.6 mm
- net Net-(R34-Pad2): track 4.00 -> 3.15 mm
- net Net-(R11-Pad1): track 25.8 -> 25.0 mm
- net Net-(R63-Pad2): track 13.5 -> 12.8 mm
- net Net-(R72-Pad2): track 26.7 -> 26.0 mm
- net LC7: track 10.1 -> 9.54 mm
- net Net-(R60-Pad2): track 19.8 -> 19.3 mm
- net Net-(R61-Pad2): track 18.7 -> 18.2 mm

Commit message: misc
Parts:
- removed ROTARY_SWITCH2: KNOB, Rotary_Encoder:RotaryEncoder_Alps_EC11E-Switch_Vertical_H20mm_CircularMountingHoles
- added R2: 0, Resistor_SMD:R_2512_6332Metric_Pad1.40x3.35mm_HandSolder, F.Cu at (386.1, 139.6)
- moved SW9 7.54 mm to (262.2, 38.9)
- moved D43 7.54 mm to (242.3, 91.7)
- moved D54 7.54 mm to (89.9, 98.4)
- moved D56 7.54 mm to (127.7, 100.9)
- moved D62 7.54 mm to (289.2, 102.4)
- moved D63 7.54 mm to (308.0, 98.4)
- moved D65 7.54 mm to (358.0, 98.4)
- moved D66 7.54 mm to (393.7, 98.4)
- moved R26 7.54 mm to (100.5, 101.6)
- moved R30 7.54 mm to (176.1, 112.4)
- moved R58 7.54 mm to (272.0, 89.7)
- moved R66 7.54 mm to (261.2, 112.4)
- moved R72 7.54 mm to (369.1, 101.6)
- moved SW59 7.54 mm to (241.9, 102.5)
- moved SW73 7.54 mm to (144.7, 114.6)
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Connections:
- net RC2 renamed Net-(R45-Pad1)
Routing:
- net RC1: track 124.8 -> 346.6 mm, vias 0 -> 1
- net LC1: track 202.8 -> 398.1 mm, vias 0 -> 1
- net RC2: track 0.00 -> 178.0 mm, vias 0 -> 1
- net RC3: track 9.72 -> 165.3 mm, vias 0 -> 1
- net RC4: track 8.32 -> 138.5 mm, vias 0 -> 1
- net LC2: track 9.28 -> 133.6 mm, vias 0 -> 1
- net LR6: track 146.0 -> 260.2 mm, vias 0 -> 2
- net RC5: track 8.32 -> 116.8 mm, vias 0 -> 1
- net LC3: track 8.83 -> 112.1 mm, vias 0 -> 1
- net RC6: track 10.5 -> 95.5 mm, vias 0 -> 1
- net LC4: track 9.60 -> 90.6 mm, vias 0 -> 1
- net RC7: track 10.7 -> 77.4 mm, vias 0 -> 1
- net LC5: track 8.99 -> 70.4 mm, vias 0 -> 1
- net LR3: track 136.4 -> 186.7 mm, vias 0 -> 1
- net LR2: track 131.3 -> 180.0 mm, vias 0 -> 1
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