File: hardware/kicad/keyboard.kicad_sch (KiCad schematic)
At the start: 185 parts, among them SW1 MX, SW10 MX, SW11 MX, SW12 MX, SW13 MX, SW14 MX, SW15 MX, SW16 MX, SW18 MX, SW19 MX, SW2 MX, SW20 MX, SW21 MX, SW22 MX, SW23 MX, SW24 MX, SW25 MX, SW26 MX, SW27 MX, SW28 MX, SW29 MX, SW3 MX, SW30 MX, SW31 MX, SW32 MX, SW33 MX, SW35 MX, SW36 MX, SW37 MX, SW38 MX, SW39 MX, SW4 MX, SW40 MX, SW41 MX, SW42 MX, SW43 MX, SW44 MX, SW45 MX, SW46 MX, SW47 MX, SW48 MX, SW49 MX, SW5 MX, SW50 MX, SW52 MX, SW53 MX, SW54 MX, SW55 MX, SW56 MX, SW57 MX, SW58 MX, SW59 MX, SW6 MX, SW60 MX, SW61 MX, SW62 MX, SW63 MX, SW64 MX, SW65 MX, SW66 MX, SW69 MX, SW7 MX, SW70 MX, SW71 MX, SW72 MX, SW73 MX, SW74 MX, SW75 MX, SW76 MX, SW77 MX, SW78 MX, SW79 MX, SW8 MX, SW80 MX, SW81 MX, SW82 MX, SW83 MX, SW84 MX, SW86 MX, SW87 MX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

Commit message: misc
Parts:
- removed U1: ESP32-S3-WROOM-1, Espressif:ESP32-S3-WROOM-1, symbol PCM_Espressif:ESP32-S3-WROOM-1
- added J1, J2: Conn_01x20_Pin, Connector_PinHeader_2.54mm:PinHeader_1x20_P2.54mm_Vertical, symbol Connector:Conn_01x20_Pin
- added R10, R11, R12, R13, R14, R15, R16, R18, R19, R20, R21, R22, R23, R25, R26, R27, R28, R29, R30, R32, R33, R34, R35, R36, R38, R39, R40, R41, R42, R43, R44, R45, R47, R48, R49, R5, R50, R51, R52, R53, R54, R56, R57, R58, R59, R6, R60, R61, R62, R63, R65, R66, R67, R68, R69, R7, R70, R71, R72, R74, R76, R77, R79, R8, R80, R81, R9: 0, Resistor_SMD:R_2512_6332Metric_Pad1.40x3.35mm_HandSolder, symbol Device:R
- added ROTARY_SWITCH2: KNOB, Rotary_Encoder:RotaryEncoder_Alps_EC11E-Switch_Vertical_H20mm_CircularMountingHoles, symbol Device:RotaryEncoder_Switch
- D1, D10, D11, D12, D13, D14, D15, D16, D18, D19, D2, D20, D21, D22, D23, D24, D25, D26, D27, D28, D29, D3, D30, D31, D32, D33, D35, D36, D37, D38, D39, D4, D40, D41, D42, D43, D44, D45, D46, D47, D48, D49, D5, D50, D52, D53, D54, D55, D56, D57, D58, D59, D6, D60, D61, D62, D63, D64, D65, D66, D69, D7, D70, D71, D72, D73, D74, D75, D76, D77, D78, D79, D8, D80, D81, D82, D83, D84, D86, D87, D88, D89, D9, D90, D91, D92, D93, D94, D95, D96, D97, D98: footprint Diode_THT:D_DO-35_SOD27_P7.62mm_Horizontal -> Diode_SMD:D_MiniMELF_Handsoldering
Connections:
- net at SW64.1: now also R61.2, R70.1
- net LC7: now reaches SW7.1
- net LC7: now also R10.1
- net RC1: now reaches SW84.1
- net RC1: now also SW16.1, SW33.1, SW50.1, SW66.1, SW98.1
- net at SW47.1: now also R52.2, R61.1
- net at SW93.1: now also R76.2
- net RC9: now reaches SW8.1
- net RC9: now also R38.1
- net at SW25.1: now also SW24.1, R10.2, R16.1
- net at SW28.1: now also R40.2, R49.1
- net LC1: now reaches SW18.1, SW35.1, SW52.1, SW69.1, SW86.1
- net LC1: now also SW1.1
- net at SW48.1: now also R53.2, R62.1
- net at SW49.1: now also R54.2, R63.1
- net RC3: now reaches SW14.1
- net RC3: now also R44.1
- net at SW77.1: now also R66.2
- net at SW43.1: now also R48.2, R57.1
- net at SW83.1: now also R72.2, R81.1
- net at SW42.1: now also R47.2, R56.1
- net at SW80.1: now also R69.2
- net at SW45.1: now also R50.2, R59.1
- net at SW29.1: now also R41.2, R50.1
- net at SW26.1: now also R38.2, R47.1
- net at SW63.1: now also R60.2, R69.1
- net at SW81.1: now also R70.2, R79.1
- net RC8: now reaches SW9.1
- net RC8: now also R39.1
- net at SW27.1: now also R39.2, R48.1
- net at SW60.1: now also R57.2, R66.1
- net RC2: now reaches SW15.1
- net RC2: now also R45.1
- net at SW61.1: now also R58.2, R67.1
- net at SW30.1: now also R42.2, R51.1
- net at SW46.1: now also R51.2, R60.1
- net at SW92.1: now also R74.2
- net at SW79.1: now also R68.2, R77.1
- net at SW59.1: now also R56.2, R65.1
- net at SW76.1: now also R65.2, R74.1
- net at SW44.1: now also R49.2, R58.1
- net at SW31.1: now also R43.2, R52.1
- net at SW62.1: now also R59.2, R68.1
- net RC4: now reaches SW13.1
- net RC4: now also R43.1
- net RC5: now reaches SW12.1
- net RC5: now also R42.1
- net at SW97.1: now also R81.2
- net RC6: now reaches SW11.1
- net RC6: now also R41.1
- net RC7: now reaches SW10.1
- net RC7: now also R40.1
- net at SW32.1: now also R45.2, R54.1
- net at SW96.1: now also R80.2
- net at SW94.1: now also R77.2
- net at SW65.1: now also R63.2, R72.1
- net at SW82.1: now also R71.2, R80.1
- net at SW95.1: now also R79.2
- net at SW78.1: now also R67.2, R76.1
- removed net C1: SW1.1, SW19.1, SW36.1, SW53.1, SW70.1, SW87.1
- removed net C2: SW2.1, SW20.1, SW37.1, SW54.1, SW71.1, SW88.1
- removed net C3: SW21.1, SW3.1, SW38.1, SW55.1, SW72.1, SW89.1
- removed net C4: SW22.1, SW39.1, SW4.1, SW56.1, SW73.1, SW90.1
- removed net C5: SW23.1, SW40.1, SW5.1, SW57.1, SW74.1, SW91.1
- removed net C6: SW24.1, SW41.1, SW58.1, SW6.1, SW75.1
- net R1 renamed RR1
- net RR1: no longer D1.1 (K), D2.1 (K), D3.1 (K), D4.1 (K), D5.1 (K), D6.1 (K), D7.1 (K)
- net R2 renamed RR2
- net RR2: no longer D18.1 (K), D19.1 (K), D20.1 (K), D21.1 (K), D22.1 (K), D23.1 (K), D24.1 (K), D25.1 (K)
- net R3 renamed RR3
- net RR3: no longer D35.1 (K), D36.1 (K), D37.1 (K), D38.1 (K), D39.1 (K), D40.1 (K), D41.1 (K)
- net R4 renamed RR4
- net RR4: no longer D52.1 (K), D53.1 (K), D54.1 (K), D55.1 (K), D56.1 (K), D57.1 (K), D58.1 (K)
- net R5 renamed RR5
- net RR5: no longer D69.1 (K), D70.1 (K), D71.1 (K), D72.1 (K), D73.1 (K), D74.1 (K), D75.1 (K)
- net R6 renamed RR6
- net RR6: no longer D86.1 (K), D87.1 (K), D88.1 (K), D89.1 (K), D90.1 (K), D91.1 (K)
- new net: R29.2, R36.1, SW74.1
- new net: R36.2, SW91.1
- new net: R22.2, R29.1, SW57.1
- new net: R23.2, R30.1, SW58.1
- new net: R30.2, SW75.1
- new net: R18.2, R25.1, SW53.1
- new net: R62.2, R71.1
- new net: R21.2, R28.1, SW56.1
- new net: R13.1, R7.2, SW21.1
- new net: R13.2, R20.1, SW38.1
- new net: R20.2, R27.1, SW55.1
- new net: R11.1, R5.2, SW19.1
- new net: R11.2, R18.1, SW36.1
- new net: R28.2, R35.1, SW73.1
- new net: R25.2, R32.1, SW70.1
- new net: R14.1, R8.2, SW22.1
- new net: R19.2, R26.1, SW54.1
- new net: R15.1, R9.2, SW23.1
- new net: R35.2, SW90.1
- new net: R16.2, R23.1, SW41.1
- new net: R14.2, R21.1, SW39.1
- new net: R27.2, R34.1, SW72.1
- new net: R34.2, SW89.1
- new net: R12.1, R6.2, SW20.1
- new net: R33.2, SW88.1
- new net: R15.2, R22.1, SW40.1
- new net: R12.2, R19.1, SW37.1
- new net: R44.2, R53.1
- new net: R32.2, SW87.1
- new net: R26.2, R33.1, SW71.1
- new net LC2: R5.1, SW2.1
- new net LC3: R6.1, SW3.1
- new net LC4: R7.1, SW4.1
- new net LC5: R8.1, SW5.1
- new net LC6: R9.1, SW6.1
- new net LR1: D1.1 (K), D2.1 (K), D3.1 (K), D4.1 (K), D5.1 (K), D6.1 (K), D7.1 (K)
- new net LR2: D18.1 (K), D19.1 (K), D20.1 (K), D21.1 (K), D22.1 (K), D23.1 (K), D24.1 (K)
- new net LR3: D35.1 (K), D36.1 (K), D37.1 (K), D38.1 (K), D39.1 (K), D40.1 (K), D41.1 (K)
- new net LR4: D52.1 (K), D53.1 (K), D54.1 (K), D55.1 (K), D56.1 (K), D57.1 (K), D58.1 (K)
- new net LR5: D69.1 (K), D70.1 (K), D71.1 (K), D72.1 (K), D73.1 (K), D74.1 (K), D75.1 (K)
- new net LR6: D25.1 (K), D86.1 (K), D87.1 (K), D88.1 (K), D89.1 (K), D90.1 (K), D91.1 (K)
Other:
- moved on the sheet: D1, D10, D11, D12, D13, D14, D15, D16, D18, D19, D2, D20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

Commit message: misc
Parts:
- removed J1, J2: Conn_01x20_Pin, Connector_PinHeader_2.54mm:PinHeader_1x20_P2.54mm_Vertical, symbol Connector:Conn_01x20_Pin
- removed ROTARY_SWITCH2: KNOB, Rotary_Encoder:RotaryEncoder_Alps_EC11E-Switch_Vertical_H20mm_CircularMountingHoles, symbol Device:RotaryEncoder_Switch
- added R2: 0, Resistor_SMD:R_2512_6332Metric_Pad1.40x3.35mm_HandSolder, symbol Device:R
Connections:
- net RC2: now also R2.2; no longer R45.1, SW15.1
- net at R81.2, SW97.1: now also R2.1
- new net: R45.1, SW15.1
Changed lines of the file:
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@@
   (junction (at 298.45 97.79) (diameter 0) (color 0 0 0 0)
   )
+  (junction (at 369.57 153.67) (diameter 0) (color 0 0 0 0)
+  )
   (junction (at 96.52 49.53) (diameter 0) (color 0 0 0 0)
   )
@@
   (junction (at 78.74 59.69) (diameter 0) (color 0 0 0 0)
   )
-  (junction (at 369.57 36.83) (diameter 0) (color 0 0 0 0)
-  )
   (junction (at 285.75 97.79) (diameter 0) (color 0 0 0 0)
   )
@@
     (stroke (width 0) (type default))
   )
+  (wire (pts (xy 369.57 153.67) (xy 369.57 165.1))
+    (stroke (width 0) (type default))
+  )
   (wire (pts (xy 356.87 101.6) (xy 356.87 118.11))
     (stroke (width 0) (type default))
@@
     (stroke (width 0) (type default))
   )
-  (wire (pts (xy 369.57 31.75) (xy 369.57 36.83))
-    (stroke (width 0) (type default))
-  )
   (wire (pts (xy 71.12 97.79) (xy 71.12 93.98))
     (stroke (width 0) (type default))
@@
     )
   )
-  (global_label "RC2" (shape input) (at 369.57 31.75 90) (fields_autoplaced)
-    (effects (font (size 1.27 1.27)) (justify left))
-    (property "Intersheetrefs" "${INTERSHEET_REFS}" (at 369.57 25.0153 90)
-      (effects (font (size 1.27 1.27)) (justify left) hide)
-    )
-  )
   (global_label "LC7" (shape input) (at 129.54 29.21 90) (fields_autoplaced)
     (effects (font (size 1.27 1.27)) (justify left))
@@
     )
   )
+  (global_label "RC2" (shape input) (at 369.57 172.72 270) (fields_autoplaced)
+    (effects (font (size 1.27 1.27)) (justify right))
+    (property "Intersheetrefs" "${INTERSHEET_REFS}" (at 369.57 179.4547 90)
+      (effects (font (size 1.27 1.27)) (justify right) hide)
+    )
+  )
   (global_label "LC4" (shape input) (at 91.44 29.21 90) (fields_autoplaced)
     (effects (font (size 1.27 1.27)) (justify left))
@@
     )
   )
-  (symbol (lib_id "Connector:Conn_01x20_Pin") (at 224.79 110.49 0) (unit 1)
-    (in_bom yes) (on_board yes) (dnp no) (fields_autoplaced)
-    (property "Reference" "J2" (at 225.425 82.55 0)
-      (effects (font (size 1.27 1.27)))
-    )
-    (property "Value" "Conn_01x20_Pin" (at 225.425 85.09 0)
-      (effects (font (size 1.27 1.27)))
-    )
-    (property "Footprint" "Connector_PinHeader_2.54mm:PinHeader_1x20_P2.54mm_Vertical" (at 224.79 110.49 0)
-      (effects (font (size 1.27 1.27)) hide)
-    )
-    (property "Datasheet" "~" (at 224.79 110.49 0)
-      (effects (font (size 1.27 1.27)) hide)
-    )
-    (pin "1")
-    (pin "10")
-    (pin "11")
-    (pin "12")
-    (pin "13")
-    (pin "14")
-    (pin "15")
-    (pin "16")
-    (pin "17")
-    (pin "18")
-    (pin "19")
-    (pin "2")
-    (pin "20")
-    (pin "3")
-    (pin "4")
-    (pin "5")
-    (pin "6")
-    (pin "7")
-    (pin "8")
-    (pin "9")
-    (instances
-      (project "esp32-s3-wroom-1-breakout"
-        (path "/03a9c855-ce75-4dbc-8ab0-a0d2cbe2834d"
-          (reference "J2") (unit 1)
-        )
-      )
-      (project "keyboard"
-        (path "/e99c776f-18bc-4796-9954-494b97c5c9e5"
-          (reference "J2") (unit 1)
-        )
-      )
-    )
-  )
   (symbol (lib_id "Device:D_Small") (at 323.85 162.56 90) (unit 1)
     (in_bom yes) (on_board yes) (dnp no)
@@
     )
   )
-  (symbol (lib_id "Device:RotaryEncoder_Switch") (at 30.48 36.83 0) (unit 1)
-    (in_bom yes) (on_board yes) (dnp no) (fields_autoplaced)
-    (property "Reference" "ROTARY_SWITCH2" (at 30.48 26.67 0)
-      (effects (font (size 1.27 1.27)))
-    )
-    (property "Value" "KNOB" (at 30.48 29.21 0)
-      (effects (font (size 1.27 1.27)))
-    )
-    (property "Footprint" "Rotary_Encoder:RotaryEncoder_Alps_EC11E-Switch_Vertical_H20mm_CircularMountingHoles" (at 26.67 32.766 0)
-      (effects (font (size 1.27 1.27)) hide)
-    )
-    (property "Datasheet" "~" (at 30.48 30.226 0)
-      (effects (font (size 1.27 1.27)) hide)
-    )
-    (pin "A")
-    (pin "B")
-    (pin "C")
-    (pin "S1")
-    (pin "S2")
-    (instances
-      (project "keyboard"
-        (path "/e99c776f-18bc-4796-9954-494b97c5c9e5"
-          (reference "ROTARY_SWITCH2") (unit 1)
-        )
-      )
-    )
-  )
   (symbol (lib_id "Device:D_Small") (at 374.65 91.44 90) (unit 1)
     (in_bom yes) (on_board yes) (dnp no)
@@
     )
   )
-  (symbol (lib_id "Connector:Conn_01x20_Pin") (at 199.39 110.49 0) (unit 1)
-    (in_bom yes) (on_board yes) (dnp no) (fields_autoplaced)
-    (property "Reference" "J1" (at 200.025 82.55 0)
-      (effects (font (size 1.27 1.27)))
-    )
-    (property "Value" "Conn_01x20_Pin" (at 200.025 85.09 0)
-      (effects (font (size 1.27 1.27)))
-    )
-    (property "Footprint" "Connector_PinHeader_2.54mm:PinHeader_1x20_P2.54mm_Vertical" (at 199.39 110.49 0)
-      (effects (font (size 1.27 1.27)) hide)
-    )
-    (property "Datasheet" "~" (at 199.39 110.49 0)
-      (effects (font (size 1.27 1.27)) hide)
-    )
-    (pin "1")
-    (pin "10")
-    (pin "11")
-    (pin "12")
-    (pin "13")
-    (pin "14")
-    (pin "15")
-    (pin "16")
-    (pin "17")
-    (pin "18")
-    (pin "19")
-    (pin "2")
-    (pin "20")
-    (pin "3")
-    (pin "4")
-    (pin "5")
-    (pin "6")
-    (pin "7")
-    (pin "8")
-    (pin "9")
-    (instances
-      (project "esp32-s3-wroom-1-breakout"
-        (path "/03a9c855-ce75-4dbc-8ab0-a0d2cbe2834d"
-          (reference "J1") (unit 1)
-        )
-      )
-      (project "keyboard"
-        (path "/e99c776f-18bc-4796-9954-494b97c5c9e5"
-          (reference "J1") (unit 1)
-        )
-      )
-    )
-  )
   (symbol (lib_id "Device:D_Small") (at 121.92 91.44 90) (unit 1)
     (in_bom yes) (on_board yes) (dnp no)
@@
         )
       )
+    )
+  )
+  (symbol (lib_id "Device:R") (at 369.57 168.91 0) (unit 1)
+    (in_bom yes) (on_board yes) (dnp no) (fields_autoplaced)
+    (property "Reference" "R2" (at 372.11 167.64 0)
+      (effects (font (size 1.27 1.27)) (justify left))
+    )
+    (property "Value" "0" (at 372.11 170.18 0)
+      (effects (font (size 1.27 1.27)) (justify left))
+    )
+    (property "Footprint" "Resistor_SMD:R_2512_6332Metric_Pad1.40x3.35mm_HandSolder" (at 367.792 168.91 90)
+      (effects (font (size 1.27 1.27)) hide)
+    )
+    (property "Datasheet" "~" (at 369.57 168.91 0)
+      (effects (font (size 1.27 1.27)) hide)
+    )
+    (pin "1")
+    (pin "2")
+    (instances
+      (project "keyboard"
+        (path "/e99c776f-18bc-4796-9954-494b97c5c9e5"
+          (reference "R2") (unit 1)
+        )
+      )
